File: rk86fdd.brd (EAGLE design)
At the start: 23 parts

Commit message: .
Parts:
- moved R1 9.92 mm to (91.4, 92.7), flipped to the bottom
- moved C1 6.48 mm to (92.7, 96.5), turned to 180 degrees
- moved R2' 3.81 mm to (29.2, 73.7), flipped to the bottom, turned to 90 degrees
- moved R2 1.80 mm to (85.1, 92.7), flipped to the bottom
Connections:
- new net N$33: DD10.1
- new net N$45: DD13.3, DD13.4
- new net N$46: DD13.5, DD13.8
- new net N$48: D9.14, DD15.8
- new net N$49: D9.2, DD10.3
- new net N$50: D9.6, DD10.13
- new net N$52: D9.11, D9.4
- new net N$53: DD14.13, DD17.9
- new net N$54: DD12.13
- new net N$55: DD12.10, DD12.12
- new net N$56: DD10.7, DD17.8
- new net N$57: DD10.12
- net B18: no longer DD14.10
- net GND: now also D9.1, D9.10, D9.15, D9.9
- net N$34: now also D9.3
- net N$9: now also DD13.2

Commit message: .
Parts:
- added R2'1, R3, R4, R5, R6, R7: 1k, rcl:R0805
- moved DD4 1.27 mm to (90.2, 31.8)
Connections:
- removed net DD6PE: DD2.1, DD2.13, DD2.22, DD6.11
- removed net N$33: DD10.1
- removed net N$52: D9.11, D9.4
- removed net N$53: DD14.13, DD17.9
- removed net N$54: DD12.13
- removed net N$55: DD12.10, DD12.12
- removed net N$56: DD10.7, DD17.8
- removed net N$57: DD10.12
- new net 1LOG: D9.11, D9.4, DD10.1, DD12.10, DD12.12, DD2.1, DD2.13, DD2.22, DD6.11, R2'1.2
- new net N$51: DD10.12, DD13.9
- net +5V: now also R2'1.1, R3.2, R4.2, R5.2, R6.2, R7.2
- net B15: now also DD10.15
- net B17: now also DD14.12
- net B18: now also DD14.10
- net B19: now also DD13.6
- net B20: now also R7.1
- net B4: now also R6.1
- net B5: now also R5.1
- net B6: now also R4.1
- net B7: now also R3.1
- net B8: now also DD12.9
- net N$23: now also D9.5, DD13.1, DD14.13, DD15.6, DD17.9
- net N$30: now also DD10.7, DD17.8
- net N$36: now also DD13.10, DD15.3
- net N$40: now also DD12.13
- net N$42: now also DD8.9
- net N$44: now also DD8.8
Routing:
- net A21: track 0.00 -> 21.7 mm
- net A24: track 0.00 -> 20.1 mm
- net A23: track 0.00 -> 20.1 mm
- net A22: track 0.00 -> 20.1 mm
- net A20: track 0.00 -> 20.1 mm
- net A11: track 0.00 -> 20.1 mm
- net A1: track 0.00 -> 20.1 mm
- net A8: track 0.00 -> 20.1 mm
- net A7: track 0.00 -> 20.1 mm
- net A6: track 0.00 -> 20.1 mm
- net A5: track 0.00 -> 20.1 mm
- net A4: track 0.00 -> 20.1 mm
- net GND: track 0.00 -> 20.1 mm
- net A9: track 0.00 -> 20.1 mm
- net A3: track 0.00 -> 20.1 mm
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