File: rk86fdd.brd (EAGLE design)
At the start: 29 parts

Commit message: .
Parts:
- added R2'': 1k, rcl:R0805
Connections:
- net B20 renamed RDDAT(20)
- net B4 renamed WPRT(4)
- net B5 renamed READY(5)
- net B6 renamed TRDO(6)
- net B7 renamed IP(7)
- new net N+: DD6.17, R2''.2
- net +5V: now also R2''.1

Commit message: .
Connections:
- net IP(7) renamed IP
- net RDDAT(20) renamed RD_DATA
- net READY(5) renamed READY
- net TRDO(6) renamed TRDO
- net WPRT(4) renamed WPRT
- removed net A11: DD1.5, DD15.13, DD4.20, DD5.20
- removed net A12: DD1.36, DD15.12
- removed net A13: DD16.2, DD16.9
- removed net A14: DD4.18
- removed net A15: DD5.18
- removed net A16: DD14.3, DD16.10, DD4.6, DD5.6
- removed net A17: DD4.5, DD5.5
- removed net A18: DD4.4, DD5.4
- removed net A19: DD4.3, DD5.3
- removed net A20: DD4.2, DD5.2
- removed net A21: DD4.1, DD5.1
- removed net A22: DD4.23, DD5.23
- removed net A23: DD4.22, DD5.22
- removed net A24: DD4.19, DD5.19
- removed net A25: DD7.14
- new net A0: DD1.9, DD16.13, DD4.8, DD5.8, X1.20
- new net CS1: DD4.18, X1.18
- new net CS2: DD5.18, X1.24
- new net CS3: DD16.2, DD16.9, X1.25
- new net D0: DD1.34, DD3.2, DD4.9, DD5.9, X1.7
- new net D1: DD1.33, DD3.5, DD4.10, DD5.10, X1.6
- new net D2: DD1.32, DD3.6, DD4.11, DD5.11, X1.19
- new net D3: DD1.31, DD3.9, DD4.13, DD5.13, X1.3
- new net D4: DD1.30, DD3.12, DD4.14, DD5.14, X1.16
- new net D5: DD1.29, DD3.15, DD4.15, DD5.15, X1.4
- new net D6: DD1.28, DD3.16, DD4.16, DD5.16, X1.17
- new net D7: DD1.27, DD3.19, DD4.17, DD5.17, X1.5
- new net OSC: DD7.14, X1.13
- new net RD: DD1.5, DD15.13, DD4.20, DD5.20, X1.2
- new net WR: DD1.36, DD15.12, X1.12
- net A1: now also DD1.8, DD16.12, DD4.7, DD5.7, X1.8; no longer DD1.34, DD3.2, DD4.9, DD5.9
- net A10: now also DD4.19, DD5.19, X1.15; no longer DD1.8, DD16.12, DD4.7, DD5.7
- net A2: now also DD14.3, DD16.10, DD4.6, DD5.6, X1.21; no longer DD1.33, DD3.5, DD4.10, DD5.10
- net A3: now also DD4.5, DD5.5, X1.9; no longer DD1.32, DD3.6, DD4.11, DD5.11
- net A4: now also DD4.4, DD5.4, X1.22; no longer DD1.31, DD3.9, DD4.13, DD5.13
- net A5: now also DD4.3, DD5.3, X1.10; no longer DD1.30, DD3.12, DD4.14, DD5.14
- net A6: now also DD4.2, DD5.2, X1.23; no longer DD1.29, DD3.15, DD4.15, DD5.15
- net A7: now also DD4.1, DD5.1, X1.11; no longer DD1.28, DD3.16, DD4.16, DD5.16
- net A8: now also DD4.23, DD5.23, X1.1; no longer DD1.27, DD3.19, DD4.17, DD5.17
- net A9: now also DD4.22, DD5.22, X1.14; no longer DD1.9, DD16.13, DD4.8, DD5.8
Routing:
- net RD: track 0.00 -> 48.6 mm
- net A7: track 20.1 -> 60.4 mm
- net D6: track 0.00 -> 40.2 mm
- net A0: track 0.00 -> 39.7 mm
- net D7: track 0.00 -> 39.3 mm
- net A6: track 20.1 -> 58.2 mm
- net A8: track 20.1 -> 57.4 mm
- net D4: track 0.00 -> 37.2 mm
- net WR: track 0.00 -> 36.9 mm
- net A9: track 20.1 -> 56.8 mm
- net D5: track 0.00 -> 35.9 mm
- net D0: track 0.00 -> 34.4 mm
- net D1: track 0.00 -> 33.9 mm
- net A5: track 20.1 -> 52.6 mm
- net A4: track 20.1 -> 52.0 mm
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
Commit message: 02
Connections:
- net CS1: now also X1.3; no longer X1.18
- net D3: now also X1.18; no longer X1.3
- net D4: now also X1.5; no longer X1.16
- net D5: now also X1.17; no longer X1.4
- net D6: now also X1.4; no longer X1.17
- net D7: now also X1.16; no longer X1.5
Routing:
- net +5V: track 0.00 -> 64.3 mm, vias 0 -> 2
- net OSC: track 0.00 -> 47.6 mm
- net D5: track 35.9 -> 77.7 mm
- net D6: track 40.2 -> 71.2 mm
- net D4: track 37.2 -> 29.5 mm
- net D3: track 31.2 -> 27.9 mm
- net D0: track 34.4 -> 36.9 mm
- net D7: track 39.3 -> 41.8 mm
- net CS1: track 24.4 -> 21.9 mm
- net D1: track 33.9 -> 31.6 mm
- net D2: track 31.9 -> 29.6 mm
- net A0: track 39.7 -> 41.6 mm

Commit message: v2
Parts:
- moved DD7 12.7 mm to (124.5, 59.1)
- moved DD8 12.7 mm to (111.8, 59.1)
- moved DD3 2.62 mm to (125.1, 29.2), turned to 270 degrees
Connections:
- net A0: now also X1.1; no longer X1.20
- net A1: now also X1.2; no longer X1.8
- net A10: now also X1.9; no longer X1.15
- net A2: now also X1.15; no longer X1.21
- net A3: now also X1.3; no longer X1.9
- net A4: now also X1.16; no longer X1.22
- net A5: now also X1.4; no longer X1.10
- net A6: now also X1.17; no longer X1.23
- net A7: now also X1.5; no longer X1.11
- net A8: now also X1.18; no longer X1.1
- net A9: now also X1.6; no longer X1.14
- net CS1: now also X1.19; no longer X1.3
- net CS2: now also X1.22; no longer X1.24
- net D0: now also X1.8; no longer X1.7
- net D1: now also X1.20; no longer X1.6
- net D2: now also X1.7; no longer X1.19
- net D3: now also X1.12; no longer X1.18
- net D4: now also X1.24; no longer X1.5
- net D5: now also X1.11; no longer X1.17
- net D6: now also X1.23; no longer X1.4
- net D7: now also X1.10; no longer X1.16
- net RD: now also X1.21; no longer X1.2
- net WR: now also X1.14; no longer X1.12
Routing:
- net OSC: track 47.6 -> 0.00 mm
- net D1: track 31.6 -> 61.3 mm
- net D2: track 29.6 -> 58.9 mm
- net D7: track 41.8 -> 60.8 mm
- net D6: track 71.2 -> 88.7 mm
- net CS3: track 17.2 -> 0.00 mm
- net D4: track 29.5 -> 45.7 mm
- net D5: track 77.7 -> 89.8 mm
- net WR: track 36.9 -> 45.7 mm
- net +5V: track 64.3 -> 56.7 mm, vias 2 -> 0
- net RD: track 48.6 -> 54.9 mm
- net A9: track 56.8 -> 50.8 mm
- net CS2: track 22.2 -> 26.7 mm
- net A0: track 41.6 -> 37.1 mm
- net D3: track 27.9 -> 31.7 mm
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
Commit message: .
Parts:
- moved R7 70.8 mm to (35.6, 86.4)
- moved R5 23.9 mm to (34.3, 7.62)
- moved R4 10.6 mm to (27.3, 25.4)
- moved R2'' 7.62 mm to (44.5, 38.1), turned to 270 degrees
- moved DD6 5.24 mm to (45.7, 33.0)
- moved R6 4.49 mm to (27.3, 19.7)
- moved R3 2.84 mm to (27.9, 41.9), turned to 270 degrees
Routing:
- net RD_DATA: track 0.00 -> 77.9 mm
- net GND: track 20.1 -> 74.5 mm
- net +5V: track 56.7 -> 100.3 mm
- net N$6: track 0.00 -> 29.6 mm
- net 1LOG: track 0.00 -> 25.2 mm
- net N$7: track 0.00 -> 23.4 mm
- net N$8: track 0.00 -> 17.9 mm
- net N$10: track 0.00 -> 15.0 mm
- net N$22: track 0.00 -> 13.8 mm
- net N$17: track 0.00 -> 13.8 mm
- net N$23: track 0.00 -> 13.5 mm
- net N$9: track 0.00 -> 12.2 mm
- net N$36: track 0.00 -> 10.8 mm
- net N$46: track 0.00 -> 9.16 mm
- net N$31: track 0.00 -> 8.03 mm
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