File: rk86fdd.sch (EAGLE design)
At the start: 23 parts

Commit message: .
Connections:
- new net N$33: DD10A.1C
- new net N$45: DD13A.O, DD13B.I0
- new net N$46: DD13B.I1, DD13C.O
- new net N$48: D9A.CLR, DD15C.O
- new net N$49: D9A.QB, DD10A.B
- new net N$50: D9A.QC, DD10A.A
- new net N$52: D9A.DN, D9A.LD
- new net N$53: DD14F.I, DD17C.I1
- new net N$54: DD12B.CLR
- new net N$55: DD12B.D, DD12B.PRE
- new net N$56: DD10A.1Y0, DD17C.I0
- new net N$57: DD10A.2Y3
- net B18: no longer DD14E.O
- net GND: now also D9A.A, D9A.B, D9A.C, D9A.D
- net N$34: now also D9A.QA
- net N$9: now also DD13A.I1
Other:
- moved on the sheet: C1, D9, DD10, DD11A, DD11B, DD12A, DD12B, DD13A, DD13B, DD13C, DD13D, DD14A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

Commit message: .
Parts:
- added R2'1, R3, R4, R5, R6, R7: 1k, rcl:R-EU_R0805
Connections:
- removed net DD6PE: DD2A.CLR, DD2A.S0, DD2A.SL, DD6A.ENC
- removed net N$33: DD10A.1C
- removed net N$52: D9A.DN, D9A.LD
- removed net N$53: DD14F.I, DD17C.I1
- removed net N$54: DD12B.CLR
- removed net N$55: DD12B.D, DD12B.PRE
- removed net N$56: DD10A.1Y0, DD17C.I0
- removed net N$57: DD10A.2Y3
- new net 1LOG: D9A.DN, D9A.LD, DD10A.1C, DD12B.D, DD12B.PRE, DD2A.CLR, DD2A.S0, DD2A.SL, DD6A.ENC, R2'1.2
- new net N$51: DD10A.2Y3, DD13C.I0
- net +5V: now also R2'1.1, R3.2, R4.2, R5.2, R6.2, R7.2
- net B15: now also DD10A.2C
- net B17: now also DD14F.O
- net B18: now also DD14E.O
- net B19: now also DD13B.O
- net B20: now also R7.1
- net B4: now also R6.1
- net B5: now also R5.1
- net B6: now also R4.1
- net B7: now also R3.1
- net B8: now also DD12B.Q
- net N$23: now also D9A.UP, DD13A.I0, DD14F.I, DD15B.O, DD17C.I1
- net N$30: now also DD10A.1Y0, DD17C.I0
- net N$36: now also DD13C.I1, DD15A.O
- net N$40: now also DD12B.CLR
- net N$42: now also DD8A.QB
- net N$44: now also DD8A.QC
Other:
- moved on the sheet: C1, D9, DD1, DD10, DD11A, DD11B, DD12A, DD12B, DD13A, DD13B, DD13C, DD13D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

Commit message: .
Parts:
- added R2'': 1k, rcl:R-EU_R0805
Connections:
- net B20 renamed RDDAT(20)
- net B4 renamed WPRT(4)
- net B5 renamed READY(5)
- net B6 renamed TRDO(6)
- net B7 renamed IP(7)
- new net N+: DD6A.7D, R2''.2
- net +5V: now also R2''.1
Other:
- note added: "Radio №2 1993"
- note added: "Radio86RK FDD controller"
- moved on the sheet: C1, D9, DD1, DD10, DD11A, DD11B, DD12A, DD12B, DD13A, DD13B, DD13C, DD13D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

Commit message: .
Connections:
- net IP(7) renamed IP
- net RDDAT(20) renamed RD_DATA
- net READY(5) renamed READY
- net TRDO(6) renamed TRDO
- net WPRT(4) renamed WPRT
- removed net A11: DD15D.I1, DD1A.RD, DD4A.!OE, DD5A.!OE
- removed net A12: DD15D.I0, DD1A.WR
- removed net A13: DD16A.I1, DD16C.I0
- removed net A14: DD4A.!CE
- removed net A15: DD5A.!CE
- removed net A16: DD14B.I, DD16C.I1, DD4A.A2, DD5A.A2
- removed net A17: DD4A.A3, DD5A.A3
- removed net A18: DD4A.A4, DD5A.A4
- removed net A19: DD4A.A5, DD5A.A5
- removed net A20: DD4A.A6, DD5A.A6
- removed net A21: DD4A.A7, DD5A.A7
- removed net A22: DD4A.A8, DD5A.A8
- removed net A23: DD4A.A9, DD5A.A9
- removed net A24: DD4A.A10, DD5A.A10
- removed net A25: DD7A.CKA
- new net A0: DD16D.I1, DD1A.A0, DD4A.A0, DD5A.A0, X1-20.M
- new net CS1: DD4A.!CE, X1-18.M
- new net CS2: DD5A.!CE, X1-24.M
- new net CS3: DD16A.I1, DD16C.I0, X1-25.M
- new net D0: DD1A.D0, DD3A.1Q, DD4A.O0, DD5A.O0, X1-7.M
- new net D1: DD1A.D1, DD3A.2Q, DD4A.O1, DD5A.O1, X1-6.M
- new net D2: DD1A.D2, DD3A.3Q, DD4A.O2, DD5A.O2, X1-19.M
- new net D3: DD1A.D3, DD3A.4Q, DD4A.O3, DD5A.O3, X1-3.M
- new net D4: DD1A.D4, DD3A.5Q, DD4A.O4, DD5A.O4, X1-16.M
- new net D5: DD1A.D5, DD3A.6Q, DD4A.O5, DD5A.O5, X1-4.M
- new net D6: DD1A.D6, DD3A.7Q, DD4A.O6, DD5A.O6, X1-17.M
- new net D7: DD1A.D7, DD3A.8Q, DD4A.O7, DD5A.O7, X1-5.M
- new net OSC: DD7A.CKA, X1-13.M
- new net RD: DD15D.I1, DD1A.RD, DD4A.!OE, DD5A.!OE, X1-2.M
- new net WR: DD15D.I0, DD1A.WR, X1-12.M
- net A1: now also DD16D.I0, DD1A.A1, DD4A.A1, DD5A.A1, X1-8.M; no longer DD1A.D0, DD3A.1Q, DD4A.O0, DD5A.O0
- net A10: now also DD4A.A10, DD5A.A10, X1-15.M; no longer DD16D.I0, DD1A.A1, DD4A.A1, DD5A.A1
- net A2: now also DD14B.I, DD16C.I1, DD4A.A2, DD5A.A2, X1-21.M; no longer DD1A.D1, DD3A.2Q, DD4A.O1, DD5A.O1
- net A3: now also DD4A.A3, DD5A.A3, X1-9.M; no longer DD1A.D2, DD3A.3Q, DD4A.O2, DD5A.O2
- net A4: now also DD4A.A4, DD5A.A4, X1-22.M; no longer DD1A.D3, DD3A.4Q, DD4A.O3, DD5A.O3
- net A5: now also DD4A.A5, DD5A.A5, X1-10.M; no longer DD1A.D4, DD3A.5Q, DD4A.O4, DD5A.O4
- net A6: now also DD4A.A6, DD5A.A6, X1-23.M; no longer DD1A.D5, DD3A.6Q, DD4A.O5, DD5A.O5
- net A7: now also DD4A.A7, DD5A.A7, X1-11.M; no longer DD1A.D6, DD3A.7Q, DD4A.O6, DD5A.O6
- net A8: now also DD4A.A8, DD5A.A8, X1-1.M; no longer DD1A.D7, DD3A.8Q, DD4A.O7, DD5A.O7
- net A9: now also DD4A.A9, DD5A.A9, X1-14.M; no longer DD16D.I1, DD1A.A0, DD4A.A0, DD5A.A0
Other:
- note added: "13 CS3 14 CS1 15 CS2 16 A2 17 A3 18 A4 19 A5 20 A6 21 A7 22 A8 23 A9 24 A10 25 OSC"
- note added: "\Шина1 Сигнал 1 D0 2 D1 3 D2 4 D3 5 D4 6 D5 7 D6 8 D7 9 A0 10 A1 11 RD 12 WR"
- note added: "Переименование сигналов"
- note added: "Шина2 Сигнал 4 WPRT 5 READY 6 TRDO 7 IP 20 RD_DATA"
- moved on the sheet: R3, R4, R5, R6, R7, X1-1, X1-10, X1-11, X1-12, X1-13, X1-14, X1-15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

Commit message: 02
Connections:
- net CS1: now also X1-3.M; no longer X1-18.M
- net D3: now also X1-18.M; no longer X1-3.M
- net D4: now also X1-5.M; no longer X1-16.M
- net D5: now also X1-17.M; no longer X1-4.M
- net D6: now also X1-4.M; no longer X1-17.M
- net D7: now also X1-16.M; no longer X1-5.M
Other:
- note added: "Смещение сигналов CS1 D3 D7 D4"

Commit message: v2
Connections:
- net A0: now also X1-1.M; no longer X1-20.M
- net A1: now also X1-2.M; no longer X1-8.M
- net A10: now also X1-9.M; no longer X1-15.M
- net A2: now also X1-15.M; no longer X1-21.M
- net A3: now also X1-3.M; no longer X1-9.M
- net A4: now also X1-16.M; no longer X1-22.M
- net A5: now also X1-4.M; no longer X1-10.M
- net A6: now also X1-17.M; no longer X1-23.M
- net A7: now also X1-5.M; no longer X1-11.M
- net A8: now also X1-18.M; no longer X1-1.M
- net A9: now also X1-6.M; no longer X1-14.M
- net CS1: now also X1-19.M; no longer X1-3.M
- net CS2: now also X1-22.M; no longer X1-24.M
- net D0: now also X1-8.M; no longer X1-7.M
- net D1: now also X1-20.M; no longer X1-6.M
- net D2: now also X1-7.M; no longer X1-19.M
- net D3: now also X1-12.M; no longer X1-18.M
- net D4: now also X1-24.M; no longer X1-5.M
- net D5: now also X1-11.M; no longer X1-17.M
- net D6: now also X1-23.M; no longer X1-4.M
- net D7: now also X1-10.M; no longer X1-16.M
- net RD: now also X1-21.M; no longer X1-2.M
- net WR: now also X1-14.M; no longer X1-12.M
Other:
- note removed: "Смещение сигналов CS1 D3 D7 D4"
- moved on the sheet: X1-1, X1-10, X1-11, X1-12, X1-13, X1-14, X1-15, X1-16, X1-17, X1-18, X1-19, X1-2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
